File: Hardware/Electronics/ProtoControlUnit/ControlUnit.sch (KiCad schematic (older format))
At the start: 17 parts, among them U1 RobotDyn_SAMD21_M0-Mini

Commit message: Encore
Parts:
- removed J?: Input from 5V boost, symbol Connector:Conn_01x03_Male
- added C?: 100uF, symbol Device:C
- added J?: Conn_01x03_Male, symbol Connector:Conn_01x03_Male
- added J?: Screw_Terminal_01x02, symbol Connector:Screw_Terminal_01x02
- added SW?: SW_DPDT_x2, symbol Switch:SW_DPDT_x2
Connections:
- net GND: now also C?.2, J?.1 (Pin_1), J?.3 (Pin_3)
- net VIN: now also C?.1, J?.2 (Pin_2), SW?.1 (A)
- net Servo_X renamed Servo_1
- net Servo_Y renamed Servo_2
- new net: J?.2 (Pin_2), SW?.2 (B)
- new net Servo_4: J?.1 (Pin_1)
- no-connect marks 6 -> 4
Other:
- moved on the sheet: C?, J?
