File: Hardware/Electronics/ControlUnit/ControlUnit.kicad_pcb (KiCad board)
At the start: 2 copper layers, 50 x 70 mm, 55 parts, among them J1 Screw_Terminal_01x02, Batt 9V, J10 Conn_01x03_Male, J11 MPU-6050/MPU-9250, J2 USB_B_Mini, J3 Conn_01x05, J4 Conn_Coaxial, J5 Conn_Coaxial, J6 Micro_SD_Card, J7 Conn_01x03_Male, J8 BME280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

Commit message: Changements...encore
Parts:
- added D3: LED, LED_SMD:LED_1206_3216Metric, F.Cu at (140.2, 79.8)
- added D4: LED, LED_SMD:LED_1206_3216Metric, F.Cu at (138.8, 70.9)
- added D5: LED, Fuse:Fuse_1206_3216Metric, F.Cu at (138.8, 73.4)
- added D6: LED, LED_SMD:LED_1206_3216Metric, F.Cu at (62.0, 110.7)
- added D7: D_Schottky, CustomLib:DIOM5436X244N, B.Cu at (137.9, 82.5)
- added D8: D_Schottky, CustomLib:DIOM5436X244N, B.Cu at (137.9, 86.6)
- added JP1: SolderJumper_2_Bridged, Jumper:SolderJumper-2_P1.3mm_Bridged_RoundedPad1.0x1.5mm, F.Cu at (67.0, 110.7)
- added Q1: BSH203, Package_TO_SOT_SMD:SOT-23, B.Cu at (144.0, 85.6)
- added R10: R, Resistor_SMD:R_0805_2012Metric, F.Cu at (135.7, 79.8)
- added R11: R, Resistor_SMD:R_0805_2012Metric, F.Cu at (69.8, 84.0)
- added R12: R, Resistor_SMD:R_0805_2012Metric, F.Cu at (70.1, 90.1)
- added R13: R, Resistor_SMD:R_0805_2012Metric, F.Cu at (61.4, 113.8)
- added R14: 10k, Resistor_SMD:R_0805_2012Metric, B.Cu at (147.6, 85.9)
- added R8: 100k, Resistor_SMD:R_0805_2012Metric, F.Cu at (141.5, 94.2)
- added R9: 100k, Resistor_SMD:R_0805_2012Metric, F.Cu at (141.5, 90.7)
- C15, C17, C18: footprint Capacitor_SMD:C_0805_2012Metric -> Capacitor_SMD:CP_Elec_6.3x7.7; moved to B.Cu
- C5, C6, R1, R2, U2, Y1: moved to B.Cu
- J10: value Conn_01x03_Male -> S3
- J7: value Conn_01x03_Male -> SX
- J9: value Conn_01x03_Male -> SY
- R7: value 100m -> 100k
- moved C16 141.3 mm to (54.1, 88.7)
- moved C8 139.0 mm to (62.2, 76.1)
- moved L1 137.2 mm to (62.0, 83.0)
- moved C14 131.1 mm to (62.2, 94.6)
- moved C11 129.1 mm to (70.6, 100.2)
- moved C1 129.1 mm to (70.9, 71.5)
- moved C2 126.0 mm to (70.4, 95.0)
- moved C3 118.4 mm to (64.5, 64.1)
- moved C13 117.5 mm to (62.2, 56.8)
- moved C7 114.4 mm to (53.6, 69.9)
- moved C12 113.8 mm to (72.1, 64.1)
- moved C19 104.0 mm to (63.2, 51.0)
- moved C4 102.0 mm to (71.1, 50.7)
- moved R6 86.3 mm to (113.6, 72.4), turned to 180 degrees
- moved C15 81.8 mm to (118.4, 105.9)
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Connections:
- C5 pad 1: Net-(C5-Pad1) -> /Vbatt
- J2 pad 1: +5VD -> Net-(D7-Pad2)
- SW1 pad 1: Net-(SW1-Pad1) -> /Vbatt
- SW1 pad 3: Net-(C5-Pad1) -> Net-(SW1-Pad3)
- U1 pad 15: Net-(U1-Pad15) -> /TX_GPS
- U1 pad 16: Net-(U1-Pad16) -> /RX_GPS
- U1 pad 26: Net-(U1-Pad26) -> /D13
- U1 pad 27: Net-(U1-Pad27) -> /CS_FLASH
- U1 pad 39: Net-(U1-Pad39) -> /TX_LED
- U1 pad 48: Net-(U1-Pad48) -> /RX_LED
- U2 pad 1: Net-(C5-Pad1) -> /Vbatt
- U5 pad 6: Net-(U5-Pad6) -> +3V3
- U5 pad 9: +3V3 -> Net-(U5-Pad9)
Routing:
- net Net-(D7-Pad2): track 0.00 -> 1.92 mm
- net /Vbatt: track 0.00 -> 1.22 mm
- net Net-(C10-Pad1): track 0.00 -> 0.71 mm
- net +5V: track 0.00 -> 0.10 mm, vias 0 -> 1
Other:
- board text added: "+"

Commit message: Encore
Parts:
- added C20: 100uF, Capacitor_SMD:CP_Elec_6.3x7.7, B.Cu at (135.0, 106.5)
- added J12: S4, Connector_PinHeader_2.54mm:PinHeader_1x03_P2.54mm_Vertical, F.Cu at (132.5, 113.0)
- added J13: Conn_01x02, Connector_PinHeader_2.54mm:PinHeader_1x02_P2.54mm_Vertical, F.Cu at (129.5, 86.5)
- C11, C13, C14, C16, C2, C3, R4, R5, R6: moved to B.Cu
- J7: value SX -> S1
- J9: value SY -> S2
- moved C16 80.7 mm to (128.2, 56.8)
- moved D6 77.0 mm to (138.5, 101.2), turned to 270 degrees
- moved R13 75.7 mm to (136.0, 101.2), turned to 270 degrees
- moved JP1 74.5 mm to (141.0, 102.0), turned to 270 degrees
- moved C19 73.9 mm to (121.5, 96.5), turned to 0 degrees
- moved C7 72.2 mm to (125.8, 67.5), turned to 270 degrees
- moved R12 72.0 mm to (140.5, 75.0), turned to 180 degrees
- moved R11 71.5 mm to (140.5, 72.8), turned to 180 degrees
- moved C14 70.3 mm to (121.5, 56.8)
- moved C13 70.0 mm to (132.2, 56.8)
- moved C1 58.3 mm to (128.0, 83.0), turned to 0 degrees
- moved C3 57.0 mm to (120.5, 74.8), turned to 0 degrees
- moved L1 56.9 mm to (118.8, 79.5)
- moved C2 55.8 mm to (120.5, 70.4), turned to 180 degrees
- moved C4 55.2 mm to (123.8, 67.5)
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Connections:
- J7 pad 1: /Servo_X -> /Servo_1
- J9 pad 1: /Servo_Y -> /Servo_2
- U1 pad 10: Net-(U1-Pad10) -> /G_LED
- U1 pad 11: Net-(U1-Pad11) -> /R_LED
- U1 pad 13: Net-(U1-Pad13) -> /Servo_1
- U1 pad 14: Net-(U1-Pad14) -> /Servo_2
- U1 pad 15: /TX_GPS -> Net-(J13-Pad2)
- U1 pad 16: /RX_GPS -> Net-(J13-Pad1)
- U1 pad 23: Net-(U1-Pad23) -> /Servo_3
- U1 pad 24: Net-(U1-Pad24) -> /Servo_4
- U1 pad 25: Net-(U1-Pad25) -> /TX_GPS
- U1 pad 27: /CS_FLASH -> /RX_GPS
- U1 pad 7: Net-(U1-Pad7) -> /Batt
- U1 pad 8: Net-(U1-Pad8) -> /BZ
- U1 pad 9: Net-(U1-Pad9) -> /B_LED
Routing:
- net Net-(C10-Pad1): track 0.71 -> 0.00 mm
- net /MOSI: track 0.00 -> 0.63 mm, vias 0 -> 1
- net Net-(J13-Pad1): track 0.00 -> 0.50 mm
- net GND: vias 0 -> 1
- net /SCK: vias 0 -> 1
- net /MISO: vias 0 -> 1
- net /CS_RAD: vias 0 -> 1
Other:
- outline, holes or cut-outs redrawn
- board text added: "vOHŇOSTROJ"

Commit message: Encore
Parts:
- added C21: 10nF, Capacitor_SMD:C_0805_2012Metric, F.Cu at (143.0, 68.8)
- added R15: 470, Resistor_SMD:R_0805_2012Metric, F.Cu at (122.5, 98.8)
- D5: footprint Fuse:Fuse_1206_3216Metric -> LED_SMD:LED_1206_3216Metric
- J13: footprint Connector_PinHeader_2.54mm:PinHeader_1x02_P2.54mm_Vertical -> CustomLib:SMD_PinHeader_01x02_2.54mm; moved to B.Cu
- J3: footprint Connector_PinHeader_2.54mm:PinHeader_1x05_P2.54mm_Vertical -> CustomLib:ProgPins_01x05_2.54mm; moved to B.Cu
- J6: footprint Connector_Card:microSD_HC_Wuerth_693072010801 -> CustomLib:microSD_HC_Molex_502774-0891
- moved J3 8.00 mm to (125.0, 45.8), turned to 90 degrees
- moved J13 5.85 mm to (127.5, 81.0), turned to 90 degrees
- moved D3 4.14 mm to (136.3, 78.4), turned to 180 degrees
- moved R10 3.44 mm to (132.3, 80.2)
- moved R3 2.00 mm to (141.0, 68.8)
- moved U6 2.00 mm to (121.5, 90.5)
- moved R7 1.25 mm to (143.0, 62.5)
- moved C19 1.00 mm to (122.5, 96.5)
- moved D6 0.75 mm to (138.5, 102.0)
- moved J6 0.71 mm to (108.5, 91.0)
- moved C1 0.50 mm to (128.0, 83.5)
- moved J5 0.35 mm to (146.5, 60.0)
- moved U5 0.26 mm to (138.8, 63.2)
- moved D5 0.16 mm to (136.3, 75.5)
Connections:
- U6 pad 3: +3V3 -> Net-(U6-Pad3)
- U6 pad 7: +3V3 -> Net-(R15-Pad2)
Routing:
- net Net-(J13-Pad1): track 0.50 -> 0.00 mm

Commit message: PCB changes
Parts:
- added G***: LOGO, CustomLib:gjna2, B.Cu at (139.5, 71.0)
- added G***: LOGO, CustomLib:gjna, F.Cu at (137.1, 83.8)
- C12: moved to B.Cu
- J3: moved to F.Cu
- moved C12 21.1 mm to (116.2, 101.0), turned to 180 degrees
- moved R12 15.2 mm to (134.8, 60.9), turned to 270 degrees
- moved R11 12.2 mm to (137.8, 60.9), turned to 270 degrees
- moved J3 11.1 mm to (125.0, 56.8), turned to 270 degrees
- moved D5 10.6 mm to (134.8, 65.0), turned to 90 degrees
- moved D4 7.79 mm to (137.9, 65.0), turned to 90 degrees
- moved L1 6.82 mm to (115.0, 73.8), turned to 0 degrees
- moved J13 5.94 mm to (123.2, 85.1), turned to 180 degrees
- moved C8 4.18 mm to (115.0, 75.7), turned to 180 degrees
- moved R2 3.66 mm to (128.9, 74.1)
- moved R1 3.07 mm to (128.9, 76.0)
- moved R13 2.15 mm to (135.9, 103.4)
- moved R10 1.80 mm to (132.3, 78.4)
- moved C19 1.50 mm to (124.0, 96.5)
- moved C13 1.46 mm to (133.5, 56.0)
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Connections:
- J3 pad 2: /SWCLK -> /RESET
- J3 pad 3: /SWDIO -> /SWCLK
- J3 pad 4: /RESET -> /SWDIO
- U1 pad 29: Net-(U1-Pad29) -> /CS_FLASH
Routing:
- net +3V3: track 0.00 -> 201.3 mm, vias 0 -> 8
- net +5V: track 0.10 -> 110.0 mm
- net /SDA: track 0.00 -> 49.4 mm, vias 0 -> 1
- net /MISO: track 0.00 -> 49.2 mm, vias 1 -> 4
- net /SCL: track 0.00 -> 48.6 mm, vias 0 -> 1
- net /SCK: track 0.00 -> 45.5 mm, vias 1 -> 2
- net /RESET: track 0.00 -> 44.9 mm
- net /MOSI: track 0.63 -> 40.8 mm, vias 1 -> 2
- net /Servo_1: track 0.00 -> 39.1 mm, vias 0 -> 2
- net /Servo_2: track 0.00 -> 37.3 mm, vias 0 -> 2
- net /Servo_3: track 0.00 -> 36.1 mm, vias 0 -> 2
- net /Servo_4: track 0.00 -> 35.6 mm, vias 0 -> 2
- net /Batt: track 0.00 -> 32.5 mm, vias 0 -> 2
- net GND: track 0.00 -> 29.7 mm, vias 1 -> 7
- net /CS_RAD: track 0.00 -> 28.3 mm
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- added copper zone on B.Cu, net GND
- added copper zone on F.Cu, net GND

Commit message: Encore
Parts:
- moved G*** 7.43 mm to (138.1, 78.3)
Routing:
- removed copper zone on B.Cu, net GND
- removed copper zone on F.Cu, net GND

Commit message: Encore
Parts:
- moved C16 3.74 mm to (127.7, 59.7), turned to 270 degrees
- moved C14 3.72 mm to (121.9, 59.7), turned to 270 degrees
- moved C6 1.37 mm to (135.2, 89.5)
- moved C13 0.71 mm to (134.2, 55.9)
- moved C11 0.40 mm to (123.2, 101.1)
- moved C5 0.30 mm to (134.1, 98.6)
- moved G*** 0.20 mm to (137.1, 84.0)
- moved C12 0.15 mm to (116.1, 101.0)
Routing:
- net +3V3: track 201.3 -> 227.1 mm, vias 8 -> 10
- net /USB_D-: track 18.2 -> 20.3 mm
- net GND: track 29.7 -> 31.4 mm, vias 7 -> 8
- net Net-(D7-Pad2): track 21.1 -> 22.1 mm
- net /USB_D+: track 19.9 -> 20.8 mm
- net /Vbatt: track 20.4 -> 19.5 mm
- net +5V: track 110.0 -> 109.1 mm
- net +5VA: track 12.2 -> 11.4 mm
- added copper zone on B.Cu, net GND
- added copper zone on F.Cu, net GND

Commit message: Encore
Other:
- board text added: "Halcyon"
- board text removed: "vOHŇOSTROJ"

Commit message: PDFs and gerber v1
Other:
- board text added: "D13"
- board text added: "RX"
- board text added: "TX"
Changed lines of the file:
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@@
   (general
     (thickness 1.6)
-    (drawings 13)
+    (drawings 16)
     (tracks 608)
     (zones 0)
@@
       (outputformat 1)
       (mirror false)
-      (drillshape 1)
+      (drillshape 0)
       (scaleselection 1)
-      (outputdirectory ""))
+      (outputdirectory "../../../../../../Desktop/"))
   )
   (net 0 "")
@@
     (descr http://www.tensility.com/pdffiles/54-00023.pdf)
     (tags "usb mini receptacle vertical")
-    (fp_text reference J2 (at 1.6 -3.7 90) (layer F.SilkS)
+    (fp_text reference J2 (at 1.71 2.088 90) (layer F.SilkS)
       (effects (font (size 1 1) (thickness 0.15)))
     )
@@
     (tags diode)
     (attr smd)
-    (fp_text reference D4 (at -3.308 0.134 90) (layer F.SilkS)
+    (fp_text reference D4 (at 2.692 -1.516 90) (layer F.SilkS)
       (effects (font (size 1 1) (thickness 0.15)))
     )
@@
     (tags diode)
     (attr smd)
-    (fp_text reference D6 (at 3 0 90) (layer F.SilkS)
+    (fp_text reference D6 (at -3.4 -0.1 90) (layer F.SilkS)
       (effects (font (size 1 1) (thickness 0.15)))
     )
@@
     (tags diode)
     (attr smd)
-    (fp_text reference D5 (at -3.3 0 90) (layer F.SilkS)
+    (fp_text reference D5 (at 2.7 -1.6 90) (layer F.SilkS)
       (effects (font (size 1 1) (thickness 0.15)))
     )
@@
     )
   )
+  (gr_text D13 (at 140.95 78.4) (layer F.SilkS)
+    (effects (font (size 1.5 1.5) (thickness 0.3)))
+  )
+  (gr_text TX (at 137.9 68.6) (layer F.SilkS)
+    (effects (font (size 1.5 1.5) (thickness 0.3)))
+  )
+  (gr_text RX (at 134.6 68.6) (layer F.SilkS)
+    (effects (font (size 1.5 1.5) (thickness 0.3)))
+  )
   (gr_line (start 140 106.25) (end 142.5 106.25) (layer F.SilkS) (width 0.15))
