File: Hardware/Electronics/ControlUnit/ControlUnit.kicad_pcb (KiCad board)
At the start: 2 copper layers, 50 x 70 mm, 77 parts, among them J1 Screw_Terminal_01x02, Batt 9V, J10 S3, J11 MPU-6050/MPU-9250, J12 S4, J13 Conn_01x02, J2 USB_B_Mini, J3 Conn_01x05, J4 Conn_Coaxial, J5 Conn_Coaxial, J6 Micro_SD_Card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

Commit message: Encore
Parts:
- added C22: 100n, Capacitor_SMD:C_0805_2012Metric, F.Cu at (139.5, 89.8)
- added Q2: , Package_TO_SOT_SMD:SOT-23, B.Cu at (140.2, 99.8)
- added R16: 10k, Resistor_SMD:R_0805_2012Metric, B.Cu at (135.9, 100.5)
- D1: value D -> D_Zener
- Q1: value BSH203 -> (none)
- U1: value ATSAMD21G18A-AF -> ATSAMD21G18A-AFT
- moved D1 10.1 mm to (140.3, 118.0), turned to 90 degrees
- moved R9 0.45 mm to (141.5, 89.8)
Connections:
- D1 pad 2: GND -> Net-(D1-Pad2)
- J1 pad 2: Net-(D1-Pad1) -> Net-(J1-Pad2)
Routing:
- net Net-(D1-Pad1): track 12.2 -> 31.3 mm
- net Net-(D1-Pad2): track 0.00 -> 10.8 mm
- net Net-(J1-Pad2): track 0.00 -> 8.23 mm
- net GND: track 31.4 -> 32.8 mm
- net /Batt: track 32.5 -> 33.8 mm

Commit message: Encore
Parts:
- removed Q1, Q2: , Package_TO_SOT_SMD:SOT-23
- removed R14, R16: 10k, Resistor_SMD:R_0805_2012Metric
- added D9: D_Schottky, CustomLib:DIOM5436X244N, B.Cu at (138.4, 81.7)
- D1: value D_Zener -> DIODE
- moved D7 8.86 mm to (145.8, 86.6)
- moved G*** 1.97 mm to (137.3, 76.5)
- moved C5 1.15 mm to (135.2, 98.9)
- moved SW1 0.55 mm to (146.1, 95.8)
- moved C6 0.41 mm to (135.3, 89.9)
- moved U2 0.41 mm to (137.8, 94.4)
- moved D8 0.38 mm to (138.3, 86.6)
- moved D1 0.10 mm to (140.2, 118.0)
Connections:
- D7 pad 1: +5V -> Net-(D7-Pad1)
- D7 pad 2: Net-(D7-Pad2) -> +5VA
- D8 pad 2: Net-(D8-Pad2) -> Net-(D7-Pad1)
- J1 pad 2: Net-(J1-Pad2) -> Net-(D1-Pad1)
- J2 pad 1: Net-(D7-Pad2) -> Net-(D9-Pad2)
- SW1 pad 2: Net-(D1-Pad1) -> Net-(D1-Pad2)
Routing:
- net Net-(D7-Pad2): track 22.1 -> 0.00 mm
- net Net-(D1-Pad1): track 31.3 -> 16.3 mm
- net Net-(D9-Pad2): track 0.00 -> 13.5 mm
- net Net-(J1-Pad2): track 8.23 -> 0.00 mm
- net +5VA: track 11.4 -> 17.3 mm
- net Net-(D8-Pad2): track 5.06 -> 0.00 mm
- net +5V: track 109.1 -> 113.0 mm
- net +3V3: track 227.1 -> 223.8 mm
- net Net-(D7-Pad1): track 0.00 -> 3.07 mm
- net GND: track 32.8 -> 34.1 mm, vias 8 -> 9
- net Net-(D1-Pad2): track 10.8 -> 9.76 mm

Commit message: Encore
Parts:
- R8: value 100k -> 33k
- R9: value 100k -> 68k

Commit message: Encore
Parts:
- moved D1 10.1 mm to (140.2, 107.9), turned to 270 degrees
Connections:
- D1 pad 1: Net-(D1-Pad1) -> Net-(D1-Pad2)
- D1 pad 2: Net-(D1-Pad2) -> Net-(D1-Pad1)
Changed lines of the file:
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@@
     (mod_text_size 1 1)
     (mod_text_width 0.15)
-    (pad_size 1.524 1.524)
-    (pad_drill 0.762)
+    (pad_size 2.2 2.2)
+    (pad_drill 1.1)
     (pad_to_mask_clearance 0.05)
     (aux_axis_origin 0 0)
@@
     )
   )
-  (module Diode_THT:D_DO-41_SOD81_P10.16mm_Horizontal (layer F.Cu)
-    (at 140.2 118 90)
-    (descr "Diode, DO-41_SOD81 series, Axial, Horizontal, pin pitch=10.16mm, , length*diameter=5.2*2.7mm^2, , http://www.diodes.com/_files/packages/DO-41%20(Plastic).pdf")
-    (tags "Diode DO-41_SOD81 series Axial Horizontal pin pitch 10.16mm  length 5.2mm diameter 2.7mm")
-    (fp_text reference D1 (at 5.2 -0.1 90) (layer F.SilkS)
-      (effects (font (size 1 1) (thickness 0.15)))
-    )
-    (fp_text value DIODE (at 5.08 2.47 90) (layer F.Fab)
-      (effects (font (size 1 1) (thickness 0.15)))
-    )
-    (fp_line (start 2.48 -1.35) (end 2.48 1.35) (layer F.Fab) (width 0.1))
-    (fp_line (start 2.48 1.35) (end 7.68 1.35) (layer F.Fab) (width 0.1))
-    (fp_line (start 7.68 1.35) (end 7.68 -1.35) (layer F.Fab) (width 0.1))
-    (fp_line (start 7.68 -1.35) (end 2.48 -1.35) (layer F.Fab) (width 0.1))
-    (fp_line (start 0 0) (end 2.48 0) (layer F.Fab) (width 0.1))
-    (fp_line (start 10.16 0) (end 7.68 0) (layer F.Fab) (width 0.1))
-    (fp_line (start 3.26 -1.35) (end 3.26 1.35) (layer F.Fab) (width 0.1))
-    (fp_line (start 3.36 -1.35) (end 3.36 1.35) (layer F.Fab) (width 0.1))
-    (fp_line (start 3.16 -1.35) (end 3.16 1.35) (layer F.Fab) (width 0.1))
-    (fp_line (start 2.36 -1.47) (end 2.36 1.47) (layer F.SilkS) (width 0.12))
-    (fp_line (start 2.36 1.47) (end 7.8 1.47) (layer F.SilkS) (width 0.12))
-    (fp_line (start 7.8 1.47) (end 7.8 -1.47) (layer F.SilkS) (width 0.12))
-    (fp_line (start 7.8 -1.47) (end 2.36 -1.47) (layer F.SilkS) (width 0.12))
-    (fp_line (start 1.34 0) (end 2.36 0) (layer F.SilkS) (width 0.12))
-    (fp_line (start 8.82 0) (end 7.8 0) (layer F.SilkS) (width 0.12))
-    (fp_line (start 3.26 -1.47) (end 3.26 1.47) (layer F.SilkS) (width 0.12))
-    (fp_line (start 3.38 -1.47) (end 3.38 1.47) (layer F.SilkS) (width 0.12))
-    (fp_line (start 3.14 -1.47) (end 3.14 1.47) (layer F.SilkS) (width 0.12))
-    (fp_line (start -1.35 -1.6) (end -1.35 1.6) (layer F.CrtYd) (width 0.05))
-    (fp_line (start -1.35 1.6) (end 11.51 1.6) (layer F.CrtYd) (width 0.05))
-    (fp_line (start 11.51 1.6) (end 11.51 -1.6) (layer F.CrtYd) (width 0.05))
-    (fp_line (start 11.51 -1.6) (end -1.35 -1.6) (layer F.CrtYd) (width 0.05))
-    (fp_text user %R (at 5.47 0 90) (layer F.Fab)
-      (effects (font (size 1 1) (thickness 0.15)))
-    )
-    (fp_text user K (at 0 -2.1 90) (layer F.Fab)
-      (effects (font (size 1 1) (thickness 0.15)))
-    )
-    (fp_text user K (at 0 -2.1 90) (layer F.SilkS)
-      (effects (font (size 1 1) (thickness 0.15)))
-    )
-    (pad 1 thru_hole rect (at 0 0 90) (size 2.2 2.2) (drill 1.1) (layers *.Cu *.Mask)
-      (net 11 "Net-(D1-Pad1)"))
-    (pad 2 thru_hole oval (at 10.16 0 90) (size 2.2 2.2) (drill 1.1) (layers *.Cu *.Mask)
-      (net 80 "Net-(D1-Pad2)"))
-    (model ${KISYS3DMOD}/Diode_THT.3dshapes/D_DO-41_SOD81_P10.16mm_Horizontal.wrl
-      (at (xyz 0 0 0))
-      (scale (xyz 1 1 1))
-      (rotate (xyz 0 0 0))
-    )
-  )
   (module CustomLib:DIOM5436X244N (layer B.Cu)
     (at 138.4 81.7)
@@
     )
   )
+  (module Diode_THT:D_DO-41_SOD81_P10.16mm_Horizontal (layer F.Cu)
+    (at 140.2 107.9 270)
+    (descr "Diode, DO-41_SOD81 series, Axial, Horizontal, pin pitch=10.16mm, , length*diameter=5.2*2.7mm^2, , http://www.diodes.com/_files/packages/DO-41%20(Plastic).pdf")
+    (tags "Diode DO-41_SOD81 series Axial Horizontal pin pitch 10.16mm  length 5.2mm diameter 2.7mm")
+    (fp_text reference D1 (at 4.5 0 90) (layer F.SilkS)
+      (effects (font (size 1 1) (thickness 0.15)))
+    )
+    (fp_text value DIODE (at 5.08 2.47 90) (layer F.Fab)
+      (effects (font (size 1 1) (thickness 0.15)))
+    )
+    (fp_line (start 11.51 -1.6) (end -1.35 -1.6) (layer F.CrtYd) (width 0.05))
+    (fp_line (start 11.51 1.6) (end 11.51 -1.6) (layer F.CrtYd) (width 0.05))
+    (fp_line (start -1.35 1.6) (end 11.51 1.6) (layer F.CrtYd) (width 0.05))
+    (fp_line (start -1.35 -1.6) (end -1.35 1.6) (layer F.CrtYd) (width 0.05))
+    (fp_line (start 3.14 -1.47) (end 3.14 1.47) (layer F.SilkS) (width 0.12))
+    (fp_line (start 3.38 -1.47) (end 3.38 1.47) (layer F.SilkS) (width 0.12))
+    (fp_line (start 3.26 -1.47) (end 3.26 1.47) (layer F.SilkS) (width 0.12))
+    (fp_line (start 8.82 0) (end 7.8 0) (layer F.SilkS) (width 0.12))
+    (fp_line (start 1.34 0) (end 2.36 0) (layer F.SilkS) (width 0.12))
+    (fp_line (start 7.8 -1.47) (end 2.36 -1.47) (layer F.SilkS) (width 0.12))
+    (fp_line (start 7.8 1.47) (end 7.8 -1.47) (layer F.SilkS) (width 0.12))
+    (fp_line (start 2.36 1.47) (end 7.8 1.47) (layer F.SilkS) (width 0.12))
+    (fp_line (start 2.36 -1.47) (end 2.36 1.47) (layer F.SilkS) (width 0.12))
+    (fp_line (start 3.16 -1.35) (end 3.16 1.35) (layer F.Fab) (width 0.1))
+    (fp_line (start 3.36 -1.35) (end 3.36 1.35) (layer F.Fab) (width 0.1))
+    (fp_line (start 3.26 -1.35) (end 3.26 1.35) (layer F.Fab) (width 0.1))
+    (fp_line (start 10.16 0) (end 7.68 0) (layer F.Fab) (width 0.1))
+    (fp_line (start 0 0) (end 2.48 0) (layer F.Fab) (width 0.1))
+    (fp_line (start 7.68 -1.35) (end 2.48 -1.35) (layer F.Fab) (width 0.1))
+    (fp_line (start 7.68 1.35) (end 7.68 -1.35) (layer F.Fab) (width 0.1))
+    (fp_line (start 2.48 1.35) (end 7.68 1.35) (layer F.Fab) (width 0.1))
+    (fp_line (start 2.48 -1.35) (end 2.48 1.35) (layer F.Fab) (width 0.1))
+    (fp_text user %R (at 5.47 0 90) (layer F.Fab)
+      (effects (font (size 1 1) (thickness 0.15)))
+    )
+    (fp_text user K (at 0 -2.1 90) (layer F.Fab)
+      (effects (font (size 1 1) (thickness 0.15)))
+    )
+    (fp_text user K (at 0 2.1 90) (layer F.SilkS)
+      (effects (font (size 1 1) (thickness 0.15)))
+    )
+    (pad 1 thru_hole rect (at 0 0 270) (size 2.2 2.2) (drill 1.1) (layers *.Cu *.Mask)
+      (net 80 "Net-(D1-Pad2)"))
+    (pad 2 thru_hole oval (at 10.16 0 270) (size 2.2 2.2) (drill 1.1) (layers *.Cu *.Mask)
+      (net 11 "Net-(D1-Pad1)"))
+    (model ${KISYS3DMOD}/Diode_THT.3dshapes/D_DO-41_SOD81_P10.16mm_Horizontal.wrl
+      (at (xyz 0 0 0))
+      (scale (xyz 1 1 1))
+      (rotate (xyz 0 0 0))
+    )
+  )

Commit message: Encore
Parts:
- removed the G*** at (137.1, 84.0)
- added G***: LOGO, CustomLib:gjnb, F.Cu at (138.4, 84.1)
- added G***: LOGO, CustomLib:Untitled, F.Cu at (118.0, 106.0)
- moved G*** 0.76 mm to (137.0, 77.2)
Routing:
- net /RESET: track 44.9 -> 44.2 mm
Other:
- board text added: "+3V3"
- board text added: "1"
- board text added: "2"
- board text added: "3"
- board text added: "4"
- board text added: "5V"
- board text added: "CS"
- board text added: "DI"
- board text added: "DO"
- board text added: "GND"
- board text added: "PWM"
- board text added: "RESET"
- board text added: "SCK"
- board text added: "SWCLK"
- board text added: "SWDIO"
- board text added: "X"
- board text removed: "Halcyon"

Commit message: Encore
Parts:
- added REF**: OSHW-Symbol_6.7x6mm_SilkScreen, Symbol:OSHW-Symbol_6.7x6mm_SilkScreen, B.Cu at (111.5, 115.2)
Routing:
- net GND: vias 9 -> 14
