File: Hardware/Electronics/ControlUnit/ControlUnit.sch (KiCad schematic (older format))
At the start: 11 parts, among them U1 RobotDyn_SAMD21_M0-Mini

Commit message: Encore
Parts:
- removed J? (x3): Conn_01x03_Male, symbol Connector:Conn_01x03_Male
- removed J?: MPU-6050, symbol Connector:Conn_01x08_Female
- removed U1: RobotDyn_SAMD21_M0-Mini, symbol CustomLib:RobotDyn_SAMD21_M0-Mini
- added BZ1: Buzzer, Buzzer_Beeper:Buzzer_12x9.5RM7.6, symbol Device:Buzzer
- added C1, C11, C13, C19, C4, C6, C8: 100nF, Capacitor_SMD:C_0805_2012Metric, symbol Device:C
- added C10: 10uF, Capacitor_SMD:C_0805_2012Metric, symbol Device:C
- added C15, C17, C18, C20: 100uF, Capacitor_SMD:CP_Elec_6.3x7.7, symbol Device:C
- added C2, C3: 12pF, Capacitor_SMD:C_0805_2012Metric, symbol Device:C
- added C5: 220nF, Capacitor_SMD:C_0805_2012Metric, symbol Device:C
- added C7, C9: 1uF, Capacitor_SMD:C_0805_2012Metric, symbol Device:C
- added D1: D, Diode_THT:D_DO-41_SOD81_P10.16mm_Horizontal, symbol Device:D
- added D2: LED_RCGB, LED_THT:LED_D5.0mm-4_RGB, symbol Device:LED_RCGB
- added D3, D4, D5, D6: LED, LED_SMD:LED_1206_3216Metric, symbol Device:LED
- added D7, D8: D_Schottky, CustomLib:DIOM5436X244N, symbol Device:D_Schottky
- added F1: 500mA, Fuse:Fuse_1206_3216Metric, symbol Device:Fuse
- added H1, H2, H3, H4: MountingHole, MountingHole:MountingHole_3.2mm_M3_DIN965_Pad, symbol Mechanical:MountingHole
- added J1: Screw_Terminal_01x02, Batt 9V, TerminalBlock_4Ucon:TerminalBlock_4Ucon_1x02_P3.50mm_Horizontal, symbol Connector:Screw_Terminal_01x02
- added J10: S3, Connector_PinHeader_2.54mm:PinHeader_1x03_P2.54mm_Vertical, symbol Connector:Conn_01x03_Male
- added J11: MPU-6050/MPU-9250, Switch:MPU-9250-4pin, symbol Connector:Conn_01x04_Female
- added J12: S4, Connector_PinHeader_2.54mm:PinHeader_1x03_P2.54mm_Vertical, symbol Connector:Conn_01x03_Male
- added J13: Conn_01x02, Connector_PinHeader_2.54mm:PinHeader_1x02_P2.54mm_Vertical, symbol Connector_Generic:Conn_01x02
- added J2: USB_B_Mini, Connector_USB:USB_Mini-B_Tensility_54-00023_Vertical_CircularHoles, symbol Connector:USB_B_Mini
- added J3: Conn_01x05, Connector_PinHeader_2.54mm:PinHeader_1x05_P2.54mm_Vertical, symbol Connector_Generic:Conn_01x05
- added J4, J5: Conn_Coaxial, Connector_Coaxial:U.FL_Hirose_U.FL-R-SMT-1_Vertical, symbol Connector:Conn_Coaxial
- added J9: S2, Connector_PinHeader_2.54mm:PinHeader_1x03_P2.54mm_Vertical, symbol Connector:Conn_01x03_Male
- added JP1: SolderJumper_2_Bridged, Jumper:SolderJumper-2_P1.3mm_Bridged_RoundedPad1.0x1.5mm, symbol Jumper:SolderJumper_2_Bridged
- added L1: 10uH, Inductor_SMD:L_0805_2012Metric, symbol Device:L
- added Q1: BSH203, Package_TO_SOT_SMD:SOT-23, symbol Transistor_FET:AO3401A
- added R1, R14, R2, R3: 10k, Resistor_SMD:R_0805_2012Metric, symbol Device:R
- added R10, R11, R12, R13: R, Resistor_SMD:R_0805_2012Metric, symbol Device:R
- added R4, R5, R6: 220, Resistor_SMD:R_0805_2012Metric, symbol Device:R
- added R7, R8, R9: 100k, Resistor_SMD:R_0805_2012Metric, symbol Device:R
- added SW1: SW_DPDT_x2, Switch:Sw1, symbol Switch:SW_DPDT_x2
- added SW2: SW_Push, CustomLib:Push_Switch_TS1107GS-5, symbol Switch:SW_Push
- added U1: ATSAMD21G18A-AF, Package_QFP:TQFP-48_7x7mm_P0.5mm, symbol MCU_Microchip_SAMD:ATSAMD21G18A-AUT
- added U2: LM340_SOT223/LM7805_5V, Package_TO_SOT_SMD:SOT-223-3_TabPin2, symbol Regulator_Linear:LM7805_TO220
- added U3: MCP1826S_3.3V, Package_TO_SOT_SMD:SOT-223-3_TabPin2, symbol Regulator_Linear:MCP1826S
- added U4: RFM69W, RF_Module:HOPERF_RFM69HW, symbol RF_Module:RFM69W
- added U5: MAX-8Q, RF_GPS:ublox_MAX, symbol RF_GPS:MAX-M8C
- added U6: W25Q32JVSS, Package_SO:SOIC-8_5.23x5.23mm_P1.27mm, symbol Memory_Flash:W25Q32JVSS
- added Y1: 32.768kHz, Crystal:Crystal_C26-LF_D2.1mm_L6.5mm_Horizontal, symbol Device:Crystal
- C12, C14, C16: renamed from C?; footprint (none) -> Capacitor_SMD:C_0805_2012Metric
- J6: renamed from J?; footprint (none) -> Connector_Card:microSD_HC_Wuerth_693072010801
- J7: renamed from J?; value Conn_01x03_Male -> S1; footprint (none) -> Connector_PinHeader_2.54mm:PinHeader_1x03_P2.54mm_Vertical
- J8: renamed from J?; footprint (none) -> CustomLib:BME280
Connections:
- net labels added: +5V, +5VA, BZ, B_LED, Batt, CS_FLASH, CS_RAD, D13, DIO0, G_LED, RESET, RX_GPS, RX_LED, R_LED, SWCLK, SWDIO, Servo_1, Servo_2, Servo_3, Servo_4, TX_GPS, TX_LED, USB_D+, USB_D-, Vbatt
- net labels removed: VIN
- wire segments 43 -> 264
- no-connect marks 7 -> 15
Other:
- note added: "D"
- note added: "EDA\nECL\nADO\nINT\nNCS\nFSYNC"
- note added: "G"
- note added: "S"
- moved on the sheet: C12, C14, C16, J6, J7, J8
