File: Hardware/Electronics/ControlUnit/ControlUnit.sch (KiCad schematic (older format))
At the start: 55 parts, among them J1 Screw_Terminal_01x02, Batt 9V, J10 Conn_01x03_Male, J11 MPU-6050/MPU-9250, J2 USB_B_Mini, J3 Conn_01x05, J4 Conn_Coaxial, J5 Conn_Coaxial, J6 Micro_SD_Card, J7 Conn_01x03_Male, J8 BME280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

Commit message: Changements...encore
Parts:
- added D3, D4, D5, D6: LED, LED_SMD:LED_1206_3216Metric, symbol Device:LED
- added D7, D8: D_Schottky, CustomLib:DIOM5436X244N, symbol Device:D_Schottky
- added JP1: SolderJumper_2_Bridged, Jumper:SolderJumper-2_P1.3mm_Bridged_RoundedPad1.0x1.5mm, symbol Jumper:SolderJumper_2_Bridged
- added Q1: BSH203, Package_TO_SOT_SMD:SOT-23, symbol Transistor_FET:AO3401A
- added R10, R11, R12, R13: R, Resistor_SMD:R_0805_2012Metric, symbol Device:R
- added R14: 10k, Resistor_SMD:R_0805_2012Metric, symbol Device:R
- added R8, R9: 100k, Resistor_SMD:R_0805_2012Metric, symbol Device:R
- C15, C17, C18: footprint Capacitor_SMD:C_0805_2012Metric -> Capacitor_SMD:CP_Elec_6.3x7.7
- J10: value Conn_01x03_Male -> S3
- J7: value Conn_01x03_Male -> SX
- J9: value Conn_01x03_Male -> SY
- R7: value 100m -> 100k
Connections:
- net labels added: Batt, D13, RX_LED, TX_LED, Vbatt
- net labels removed: +5VD
- wire segments 210 -> 245
- no-connect marks 14 -> 15
Other:
- note added: "D"
- note added: "G"
- note added: "S"
- moved on the sheet: C10, C5, C6, C9, D1, F1, J1, J2, J3, R3, R7, SW1A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

Commit message: Encore
Parts:
- added C20: 100uF, Capacitor_SMD:CP_Elec_6.3x7.7, symbol Device:C
- added J12: S4, Connector_PinHeader_2.54mm:PinHeader_1x03_P2.54mm_Vertical, symbol Connector:Conn_01x03_Male
- added J13: Conn_01x02, Connector_PinHeader_2.54mm:PinHeader_1x02_P2.54mm_Vertical, symbol Connector_Generic:Conn_01x02
- J7: value SX -> S1
- J9: value SY -> S2
Connections:
- net Servo_X is gone; now on net Servo_1: J7.1 (Pin_1)
- net Servo_Y is gone; now on net Servo_2: J9.1 (Pin_1)
- net +5V: now also C20.1, J12.2 (Pin_2)
- net BZ: now also U1.8 (PB09)
- net B_LED: now also U1.9 (PA04)
- net Batt: now also U1.7 (PB08)
- net CS_FLASH: no longer U1.27 (PA18)
- net GND: now also C20.2, J12.3 (Pin_3)
- net G_LED: now also U1.10 (PA05)
- net RX_GPS: now also U1.27 (PA18); no longer U1.16 (PA11)
- net R_LED: now also U1.11 (PA06)
- net Servo_3: now also U1.23 (PA14)
- net TX_GPS: now also U1.25 (PA16); no longer U1.15 (PA10)
- net Servo_1: now reaches U1.13 (PA08)
- net Servo_2: now reaches U1.14 (PA09)
- net Servo_4: now reaches U1.24 (PA15)
- net Servo_4: now also J12.1 (Pin_1)
- new net: J13.2 (Pin_2), U1.15 (PA10)
- new net: J13.1 (Pin_1), U1.16 (PA11)
Other:
- moved on the sheet: C18, J10

Commit message: Encore
Parts:
- added C21: 10nF, Capacitor_SMD:C_0805_2012Metric, symbol Device:C
- added R15: 470, Resistor_SMD:R_0805_2012Metric, symbol Device:R
- J13: footprint Connector_PinHeader_2.54mm:PinHeader_1x02_P2.54mm_Vertical -> CustomLib:SMD_PinHeader_01x02_2.54mm
- J3: footprint Connector_PinHeader_2.54mm:PinHeader_1x05_P2.54mm_Vertical -> CustomLib:ProgPins_01x05_2.54mm
- J6: footprint Connector_Card:microSD_HC_Wuerth_693072010801 -> CustomLib:microSD_HC_Molex_502774-0891
Connections:
- net +3V3: now also R15.1; no longer U6.3 (IO2), U6.7 (IO3)
- net GND: now also C21.2
- net RESET: now also C21.1
- new net: R15.2, U6.7 (IO3)
Other:
- moved on the sheet: C19, R3, R7, SW2
Changed lines of the file:
@@
 U 1 1 604D9C4E
 P 12650 4450
-F 0 "C14" H 12450 4500 50  0000 L CNN
+F 0 "C14" H 12350 4500 50  0000 L CNN
 F 1 "100nF" H 12300 4400 50  0000 L CNN
 F 2 "Capacitor_SMD:C_0805_2012Metric" H 12688 4300 50  0001 C CNN
@@
 F 0 "J6" H 11750 8117 50  0000 C CNN
 F 1 "Micro_SD_Card" H 11750 8026 50  0000 C CNN
-F 2 "Connector_Card:microSD_HC_Wuerth_693072010801" H 12950 7700 50  0001 C CNN
+F 2 "CustomLib:microSD_HC_Molex_502774-0891" H 12950 7700 50  0001 C CNN
 F 3 "http://katalog.we-online.de/em/datasheet/693072010801.pdf" H 11800 7400 50  0001 C CNN
 	1    11800 7400
@@
 U 1 1 604EA756
 P 14150 4450
-F 0 "C16" H 13950 4500 50  0000 L CNN
+F 0 "C16" H 13850 4500 50  0000 L CNN
 F 1 "100nF" H 13800 4400 50  0000 L CNN
 F 2 "Capacitor_SMD:C_0805_2012Metric" H 14188 4300 50  0001 C CNN
@@
 	14700 7300 14850 7300
 Wire Wire Line
-	14700 7500 15150 7500
-Wire Wire Line
 	14700 7600 15150 7600
-Wire Wire Line
-	15150 7600 15150 7500
-Connection ~ 15150 7500
 $Comp
 L power:+3V3 #PWR059
 U 1 1 604E9644
-P 15150 6800
-F 0 "#PWR059" H 15150 6650 50  0001 C CNN
-F 1 "+3V3" H 15165 6973 50  0000 C CNN
-F 2 "" H 15150 6800 50  0001 C CNN
-F 3 "" H 15150 6800 50  0001 C CNN
-	1    15150 6800
+P 15450 6850
+F 0 "#PWR059" H 15450 6700 50  0001 C CNN
+F 1 "+3V3" H 15465 7023 50  0000 C CNN
+F 2 "" H 15450 6850 50  0001 C CNN
+F 3 "" H 15450 6850 50  0001 C CNN
+	1    15450 6850
 	1    0    0    -1
 $EndComp
 Wire Wire Line
 	14200 6900 15150 6900
-Wire Wire Line
-	15150 6900 15150 7500
 Text Label 13300 7300 0    50   ~ 0
 CS_FLASH
@@
 L Device:C C19
 U 1 1 604F503D
-P 15150 7750
-F 0 "C19" H 15300 7800 50  0000 L CNN
-F 1 "100nF" H 15300 7700 50  0000 L CNN
-F 2 "Capacitor_SMD:C_0805_2012Metric" H 15188 7600 50  0001 C CNN
-F 3 "~" H 15150 7750 50  0001 C CNN
-	1    15150 7750
+P 15450 7100
+F 0 "C19" H 15600 7150 50  0000 L CNN
+F 1 "100nF" H 15600 7050 50  0000 L CNN
+F 2 "Capacitor_SMD:C_0805_2012Metric" H 15488 6950 50  0001 C CNN
+F 3 "~" H 15450 7100 50  0001 C CNN
+	1    15450 7100
 	1    0    0    -1
 $EndComp
@@
 L power:GND #PWR060
 U 1 1 604F5043
-P 15150 8000
-F 0 "#PWR060" H 15150 7750 50  0001 C CNN
-F 1 "GND" H 15155 7827 50  0000 C CNN
-F 2 "" H 15150 8000 50  0001 C CNN
-F 3 "" H 15150 8000 50  0001 C CNN
-	1    15150 8000
-	1    0    0    -1
-$EndComp
-Wire Wire Line
-	15150 7900 15150 8000
+P 15450 7350
+F 0 "#PWR060" H 15450 7100 50  0001 C CNN
+F 1 "GND" H 15455 7177 50  0000 C CNN
+F 2 "" H 15450 7350 50  0001 C CNN
+F 3 "" H 15450 7350 50  0001 C CNN
+	1    15450 7350
+	1    0    0    -1
+$EndComp
+Wire Wire Line
+	15450 7250 15450 7350
 $Comp
 L MCU_Microchip_SAMD:ATSAMD21G18A-AUT U1
@@
 	1    0    0    -1
 $EndComp
-Connection ~ 15150 7600
 $Comp
 L RF_GPS:MAX-M8C U5
@@
 F 0 "J3" H 9000 10450 50  0000 L CNN
 F 1 "Conn_01x05" H 8950 10350 50  0000 L CNN
-F 2 "Connector_PinHeader_2.54mm:PinHeader_1x05_P2.54mm_Vertical" H 9000 10000 50  0001 C CNN
+F 2 "CustomLib:ProgPins_01x05_2.54mm" H 9000 10000 50  0001 C CNN
 F 3 "~" H 9000 10000 50  0001 C CNN
 	1    9000 10000
@@
 L Switch:SW_Push SW2
 U 1 1 605D4BE8
-P 8950 9100
-F 0 "SW2" H 8950 9385 50  0000 C CNN
-F 1 "SW_Push" H 8950 9294 50  0000 C CNN
-F 2 "CustomLib:Push_Switch_TS1107GS-5" H 8950 9300 50  0001 C CNN
-F 3 "~" H 8950 9300 50  0001 C CNN
-	1    8950 9100
-	1    0    0    -1
-$EndComp
-Wire Wire Line
-	8750 9100 8550 9100
-Text Label 8200 9100 0    50   ~ 0
+P 8900 8850
+F 0 "SW2" H 8900 9135 50  0000 C CNN
+F 1 "SW_Push" H 8900 9044 50  0000 C CNN
+F 2 "CustomLib:Push_Switch_TS1107GS-5" H 8900 9050 50  0001 C CNN
+F 3 "~" H 8900 9050 50  0001 C CNN
+	1    8900 8850
+	1    0    0    -1
+$EndComp
+Wire Wire Line
+	8700 8850 8500 8850
+Text Label 8150 8850 0    50   ~ 0
 RESET
 $Comp
 L power:GND #PWR033
 U 1 1 6060523C
-P 9650 9150
-F 0 "#PWR033" H 9650 8900 50  0001 C CNN
-F 1 "GND" H 9655 8977 50  0000 C CNN
-F 2 "" H 9650 9150 50  0001 C CNN
-F 3 "" H 9650 9150 50  0001 C CNN
-	1    9650 9150
+P 9600 8900
+F 0 "#PWR033" H 9600 8650 50  0001 C CNN
+F 1 "GND" H 9605 8727 50  0000 C CNN
+F 2 "" H 9600 8900 50  0001 C CNN
+F 3 "" H 9600 8900 50  0001 C CNN
+	1    9600 8900
 	1    0    0    -1
 $EndComp
@@
 L Device:R R3
 U 1 1 607354D9
-P 8550 8850
-F 0 "R3" H 8620 8896 50  0000 L CNN
-F 1 "10k" H 8620 8805 50  0000 L CNN
-F 2 "Resistor_SMD:R_0805_2012Metric" V 8480 8850 50  0001 C CNN
-F 3 "~" H 8550 8850 50  0001 C CNN
-	1    8550 8850
+P 8500 8600
+F 0 "R3" H 8570 8646 50  0000 L CNN
+F 1 "10k" H 8570 8555 50  0000 L CNN
+F 2 "Resistor_SMD:R_0805_2012Metric" V 8430 8600 50  0001 C CNN
+F 3 "~" H 8500 8600 50  0001 C CNN
+	1    8500 8600
 	1    0    0    -1
 $EndComp
@@
 L power:+3V3 #PWR06
 U 1 1 607364AD
-P 8550 8650
-F 0 "#PWR06" H 8550 8500 50  0001 C CNN
-F 1 "+3V3" H 8565 8823 50  0000 C CNN
-F 2 "" H 8550 8650 50  0001 C CNN
-F 3 "" H 8550 8650 50  0001 C CNN
-	1    8550 8650
-	1    0    0    -1
-$EndComp
-Wire Wire Line
-	8550 8650 8550 8700
+P 8500 8400
+F 0 "#PWR06" H 8500 8250 50  0001 C CNN
+F 1 "+3V3" H 8515 8573 50  0000 C CNN
+F 2 "" H 8500 8400 50  0001 C CNN
+F 3 "" H 8500 8400 50  0001 C CNN
+	1    8500 8400
+	1    0    0    -1
+$EndComp
+Wire Wire Line
+	8500 8400 8500 8450
 Wire Wire Line
 	2500 4650 1100 4650
@@
 BZ
 Wire Wire Line
-	15150 6800 15150 6900
-Connection ~ 15150 6900
+	15450 6850 15450 6900
 $Comp
 L Connector:USB_B_Mini J2
@@
 L Device:R R7
 U 1 1 6057AD29
-P 9400 9100
-F 0 "R7" V 9193 9100 50  0000 C CNN
-F 1 "100k" V 9284 9100 50  0000 C CNN
-F 2 "Resistor_SMD:R_0805_2012Metric" V 9330 9100 50  0001 C CNN
-F 3 "~" H 9400 9100 50  0001 C CNN
-	1    9400 9100
+P 9350 8850
+F 0 "R7" V 9143 8850 50  0000 C CNN
+F 1 "100k" V 9234 8850 50  0000 C CNN
+F 2 "Resistor_SMD:R_0805_2012Metric" V 9280 8850 50  0001 C CNN
+F 3 "~" H 9350 8850 50  0001 C CNN
+	1    9350 8850
 	0    1    1    0
 $EndComp
 Wire Wire Line
-	9650 9100 9650 9150
-Wire Wire Line
-	9550 9100 9650 9100
-Wire Wire Line
-	9150 9100 9250 9100
+	9600 8850 9600 8900
+Wire Wire Line
+	9500 8850 9600 8850
+Wire Wire Line
+	9100 8850 9200 8850
 $Comp
 L power:+3V3 #PWR011
@@
 D13
 Wire Wire Line
-	8550 9000 8550 9100
-Connection ~ 8550 9100
-Wire Wire Line
-	8550 9100 8200 9100
+	8500 8750 8500 8850
+Connection ~ 8500 8850
+Wire Wire Line
+	8500 8850 8150 8850
 Text Label 4700 2650 0    50   ~ 0
 Batt
@@
 F 0 "J13" H 2000 3450 50  0000 C CNN
 F 1 "Conn_01x02" H 2200 3550 50  0000 C CNN
-F 2 "Connector_PinHeader_2.54mm:PinHeader_1x02_P2.54mm_Vertical" H 1850 3550 50  0001 C CNN
+F 2 "CustomLib:SMD_PinHeader_01x02_2.54mm" H 1850 3550 50  0001 C CNN
 F 3 "~" H 1850 3550 50  0001 C CNN
 	1    1850 3550
@@
 	4500 2650 4700 2650
 Wire Wire Line
+	2500 2850 2150 2850
+Wire Wire Line
+	2500 2950 2150 2950
+Wire Wire Line
+	2500 3050 2150 3050
+Wire Wire Line
+	2500 3850 2150 3850
+Wire Wire Line
+	2500 4250 2150 4250
+Wire Wire Line
+	2500 4050 2150 4050
+$Comp
+L Device:R R15
+U 1 1 6065A09E
+P 15150 7350
+F 0 "R15" H 15220 7396 50  0000 L CNN
+F 1 "470" H 15220 7305 50  0000 L CNN
+F 2 "Resistor_SMD:R_0805_2012Metric" V 15080 7350 50  0001 C CNN
+F 3 "~" H 15150 7350 50  0001 C CNN
+	1    15150 7350
+	1    0    0    -1
+$EndComp
+Wire Wire Line
+	15150 7600 15150 7500
+Wire Wire Line
+	15150 7200 15150 6900
+Connection ~ 15150 6900
+Wire Wire Line
+	15150 6900 15450 6900
+Connection ~ 15450 6900
+Wire Wire Line
+	15450 6900 15450 6950
+Wire Wire Line
 	4500 2750 4700 2750
 Wire Wire Line
-	2500 2850 2150 2850
-Wire Wire Line
-	2500 2950 2150 2950
-Wire Wire Line
-	2500 3050 2150 3050
-Wire Wire Line
-	2500 3850 2150 3850
-Wire Wire Line
-	2500 4250 2150 4250
-Wire Wire Line
-	2500 4050 2150 4050
+	8500 8850 8500 8950
+$Comp
+L Device:C C21
+U 1 1 606E17B0
+P 8500 9100
+F 0 "C21" H 8615 9146 50  0000 L CNN
+F 1 "10nF" H 8615 9055 50  0000 L CNN
+F 2 "Capacitor_SMD:C_0805_2012Metric" H 8538 8950 50  0001 C CNN
+F 3 "~" H 8500 9100 50  0001 C CNN
+	1    8500 9100
+	1    0    0    -1
+$EndComp
+Wire Wire Line
+	8500 9250 8500 9300
+$Comp
+L power:GND #PWR0110
+U 1 1 6070E5D7
+P 8500 9300
+F 0 "#PWR0110" H 8500 9050 50  0001 C CNN
+F 1 "GND" H 8650 9250 50  0000 C CNN
+F 2 "" H 8500 9300 50  0001 C CNN
+F 3 "" H 8500 9300 50  0001 C CNN
+	1    8500 9300
+	1    0    0    -1
+$EndComp
 $EndSCHEMATC

Commit message: PCB changes
Connections:
- net CS_FLASH: now also U1.29 (PA20)
- net RESET: now also J3.2 (Pin_2); no longer J3.4 (Pin_4)
- net SWCLK: now also J3.3 (Pin_3); no longer J3.2 (Pin_2)
- net SWDIO: now also J3.4 (Pin_4); no longer J3.3 (Pin_3)
- no-connect marks 15 -> 24
Other:
- note added: "Flash chip"
- note added: "GNSS module"
- note added: "Microcontroller"
- note added: "Mounting holes"
- note added: "Optional devices"
- note added: "Power management"
- note added: "Programming and reset"
- note added: "Sensors"
- note added: "Servos"
- note added: "State indicators"
- note added: "Storage devices"
- note added: "Transceiver"
- note added: "microSD card slot"
- moved on the sheet: BZ1, C1, C10, C11, C12, C13, C14, C15, C16, C17, C18, C19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

Commit message: Encore
Parts:
- U1: value ATSAMD21G18A-AF -> ATSAMD21G18A-AFT
Changed lines of the file:
@@
 P 3700 4400
 F 0 "U1" H 2950 2600 50  0000 C CNN
-F 1 "ATSAMD21G18A-AF" H 3000 2500 50  0000 C CNN
+F 1 "ATSAMD21G18A-AFT" H 3000 2500 50  0000 C CNN
 F 2 "Package_QFP:TQFP-48_7x7mm_P0.5mm" H 2750 2650 50  0001 C CNN
 F 3 "http://ww1.microchip.com/downloads/en/DeviceDoc/SAM_D21_DA1_Family_Data%20Sheet_DS40001882E.pdf" H 3700 5400 50  0001 C CNN

Commit message: Encore
Changed lines of the file:
@@
 U 1 1 604C3592
 P 12900 2000
-F 0 "J7" H 13150 2350 50  0000 C CNN
-F 1 "S1" H 13150 2250 50  0000 C CNN
+F 0 "J7" H 12950 2350 50  0000 C CNN
+F 1 "S1" H 12950 2250 50  0000 C CNN
 F 2 "Connector_PinHeader_2.54mm:PinHeader_1x03_P2.54mm_Vertical" H 12900 2000 50  0001 C CNN
 F 3 "~" H 12900 2000 50  0001 C CNN
@@
 U 1 1 60669239
 P 14200 2000
-F 0 "J9" H 14450 2350 50  0000 C CNN
-F 1 "S2" H 14450 2250 50  0000 C CNN
+F 0 "J9" H 14250 2350 50  0000 C CNN
+F 1 "S2" H 14250 2250 50  0000 C CNN
 F 2 "Connector_PinHeader_2.54mm:PinHeader_1x03_P2.54mm_Vertical" H 14200 2000 50  0001 C CNN
 F 3 "~" H 14200 2000 50  0001 C CNN
@@
 U 1 1 60672E64
 P 12900 2950
-F 0 "J10" H 13150 3300 50  0000 C CNN
-F 1 "S3" H 13150 3200 50  0000 C CNN
+F 0 "J10" H 12950 3300 50  0000 C CNN
+F 1 "S3" H 12950 3200 50  0000 C CNN
 F 2 "Connector_PinHeader_2.54mm:PinHeader_1x03_P2.54mm_Vertical" H 12900 2950 50  0001 C CNN
 F 3 "~" H 12900 2950 50  0001 C CNN
@@
 U 1 1 605A3804
 P 14200 2950
-F 0 "J12" H 14450 3300 50  0000 C CNN
-F 1 "S4" H 14450 3200 50  0000 C CNN
+F 0 "J12" H 14250 3300 50  0000 C CNN
+F 1 "S4" H 14250 3200 50  0000 C CNN
 F 2 "Connector_PinHeader_2.54mm:PinHeader_1x03_P2.54mm_Vertical" H 14200 2950 50  0001 C CNN
 F 3 "~" H 14200 2950 50  0001 C CNN

Commit message: Encore
Parts:
- removed D1: D, Diode_THT:D_DO-41_SOD81_P10.16mm_Horizontal, symbol Device:D
- added C22: 100n, symbol Device:C
- added D1: D_Zener, symbol Device:D_Zener
- added Q2: (no value), Package_TO_SOT_SMD:SOT-23, symbol Transistor_FET:BS250
- added R16: R, symbol Device:R
- Q1: value BSH203 -> (none)
Connections:
- net Batt: now also C22.1
- net GND: now also C22.2, R16.2
- net at SW1.2 (B): now also D1.1 (K), Q2.3 (S); no longer J1.2 (Pin_2)
- new net: J1.2 (Pin_2), Q2.1 (D)
- new net: D1.2 (A), Q2.2 (G), R16.1
Other:
- moved on the sheet: J1, SW1A
Changed lines of the file:
@@
 Comment4 ""
 $EndDescr
-Wire Wire Line
-	1700 8100 2050 8100
-Wire Wire Line
-	2050 8100 2050 8200
-$Comp
-L power:GND #PWR05
-U 1 1 604B9A62
-P 2050 8200
-F 0 "#PWR05" H 2050 7950 50  0001 C CNN
-F 1 "GND" H 2055 8027 50  0000 C CNN
-F 2 "" H 2050 8200 50  0001 C CNN
-F 3 "" H 2050 8200 50  0001 C CNN
-	1    2050 8200
-	1    0    0    -1
-$EndComp
 $Comp
 L Connector:Conn_01x03_Male J7
@@
 $EndComp
 $Comp
-L Device:D D1
-U 1 1 6054242C
-P 2250 8200
-F 0 "D1" V 2204 8280 50  0000 L CNN
-F 1 "D" V 2295 8280 50  0000 L CNN
-F 2 "Diode_THT:D_DO-41_SOD81_P10.16mm_Horizontal" H 2250 8200 50  0001 C CNN
-F 3 "~" H 2250 8200 50  0001 C CNN
-	1    2250 8200
-	0    1    1    0
-$EndComp
-Wire Wire Line
-	2250 8350 2250 8400
-$Comp
 L power:GND #PWR08
 U 1 1 6054633D
-P 2250 8400
-F 0 "#PWR08" H 2250 8150 50  0001 C CNN
-F 1 "GND" H 2255 8227 50  0000 C CNN
-F 2 "" H 2250 8400 50  0001 C CNN
-F 3 "" H 2250 8400 50  0001 C CNN
-	1    2250 8400
-	1    0    0    -1
-$EndComp
-Wire Wire Line
-	2250 8000 2250 8050
-Connection ~ 2250 8000
-Wire Wire Line
-	2250 8000 2400 8000
-Wire Wire Line
-	1700 8000 2250 8000
+P 1450 8750
+F 0 "#PWR08" H 1450 8500 50  0001 C CNN
+F 1 "GND" H 1455 8577 50  0000 C CNN
+F 2 "" H 1450 8750 50  0001 C CNN
+F 3 "" H 1450 8750 50  0001 C CNN
+	1    1450 8750
+	1    0    0    -1
+$EndComp
 $Comp
 L Device:Fuse F1
@@
 L Connector:Screw_Terminal_01x02 J1
 U 1 1 606C8AB5
-P 1500 8100
-F 0 "J1" H 1418 7775 50  0000 C CNN
-F 1 "Screw_Terminal_01x02, Batt 9V" H 1418 7866 50  0000 C CNN
-F 2 "TerminalBlock_4Ucon:TerminalBlock_4Ucon_1x02_P3.50mm_Horizontal" H 1500 8100 50  0001 C CNN
-F 3 "~" H 1500 8100 50  0001 C CNN
-	1    1500 8100
+P 1150 8100
+F 0 "J1" H 1100 7750 50  0000 C CNN
+F 1 "Screw_Terminal_01x02, Batt 9V" H 700 7850 50  0000 C CNN
+F 2 "TerminalBlock_4Ucon:TerminalBlock_4Ucon_1x02_P3.50mm_Horizontal" H 1150 8100 50  0001 C CNN
+F 3 "~" H 1150 8100 50  0001 C CNN
+	1    1150 8100
 	-1   0    0    1
 $EndComp
@@
 Text Label 4900 3000 0    50   ~ 0
 Batt
-Text Label 5100 9550 0    50   ~ 0
+Text Label 4850 9550 0    50   ~ 0
 Batt
 $Comp
@@
 	1    0    0    -1
 $EndComp
-Text Label 3200 7750 0    50   ~ 0
+Text Label 3350 7750 0    50   ~ 0
 Vbatt
 Text Label 5350 9100 0    50   ~ 0
@@
 Wire Wire Line
 	5350 9500 5350 9550
-Wire Wire Line
-	5350 9550 5100 9550
 Connection ~ 5350 9550
 Wire Wire Line
@@
 P 3100 9850
 F 0 "Q1" V 3100 10000 50  0000 L CNN
-F 1 "BSH203" V 3000 10000 50  0000 L CNN
+F 1 " " V 3000 10000 50  0000 L CNN
 F 2 "Package_TO_SOT_SMD:SOT-23" H 3300 9775 50  0001 L CIN
 F 3 "http://www.aosmd.com/pdfs/datasheet/AO3401A.pdf" H 3100 9850 50  0001 L CNN
@@
 	1900 9300 2500 9300
 Wire Wire Line
-	2800 7900 3200 7900
-Wire Wire Line
-	3200 7900 3200 7750
-Connection ~ 3200 7900
-Wire Wire Line
-	3200 7900 3650 7900
+	3150 7900 3350 7900
+Wire Wire Line
+	3350 7900 3350 7750
+Connection ~ 3350 7900
+Wire Wire Line
+	3350 7900 3650 7900
 Wire Wire Line
 	15200 1950 15200 2000
@@
 L Switch:SW_DPDT_x2 SW1
 U 1 1 6054C740
-P 2600 8000
-F 0 "SW1" H 2600 8285 50  0000 C CNN
-F 1 "SW_DPDT_x2" H 2600 8194 50  0000 C CNN
-F 2 "Switch:Sw1" H 2600 8000 50  0001 C CNN
-F 3 "~" H 2600 8000 50  0001 C CNN
-	1    2600 8000
+P 2950 8000
+F 0 "SW1" H 2950 8285 50  0000 C CNN
+F 1 "SW_DPDT_x2" H 2950 8194 50  0000 C CNN
+F 2 "Switch:Sw1" H 2950 8000 50  0001 C CNN
+F 3 "~" H 2950 8000 50  0001 C CNN
+	1    2950 8000
 	1    0    0    -1
 $EndComp
@@
 NoConn ~ 2700 4900
 NoConn ~ 2700 4700
-NoConn ~ 2800 8100
+NoConn ~ 3150 8100
 Wire Wire Line
 	7400 2050 7400 1950
@@
 Text Notes 9600 7350 0    50   ~ 10
 State indicators
+$Comp
+L Device:D_Zener D1
+U 1 1 608DBB45
+P 2550 8150
+F 0 "D1" V 2504 8230 50  0000 L CNN
+F 1 "D_Zener" V 2595 8230 50  0000 L CNN
+F 2 "" H 2550 8150 50  0001 C CNN
+F 3 "~" H 2550 8150 50  0001 C CNN
+	1    2550 8150
+	0    1    1    0
+$EndComp
+$Comp
+L Transistor_FET:BS250 Q2
+U 1 1 6091F04D
+P 2250 8100
+F 0 "Q2" V 2500 7900 50  0000 C CNN
+F 1 " " V 2501 8100 50  0000 C CNN
+F 2 "Package_TO_SOT_SMD:SOT-23" H 2450 8025 50  0001 L CIN
+F 3 "http://www.vishay.com/docs/70209/70209.pdf" H 2250 8100 50  0001 L CNN
+	1    2250 8100
+	0    -1   -1   0
+$EndComp
+Wire Wire Line
+	1350 8000 2050 8000
+Wire Wire Line
+	1350 8100 1450 8100
+$Comp
+L Device:R R16
+U 1 1 609CD907
+P 2250 8500
+F 0 "R16" H 2320 8546 50  0000 L CNN
+F 1 "R" H 2320 8455 50  0000 L CNN
+F 2 "" V 2180 8500 50  0001 C CNN
+F 3 "~" H 2250 8500 50  0001 C CNN
+	1    2250 8500
+	1    0    0    -1
+$EndComp
+Wire Wire Line
+	2450 8000 2550 8000
+Connection ~ 2550 8000
+Wire Wire Line
+	2550 8000 2750 8000
+Wire Wire Line
+	1450 8100 1450 8700
+Wire Wire Line
+	2250 8300 2250 8350
+Wire Wire Line
+	2550 8300 2550 8350
+Wire Wire Line
+	2550 8350 2250 8350
+Connection ~ 2250 8350
+Wire Wire Line
+	2250 8650 2250 8700
+Wire Wire Line
+	2250 8700 1450 8700
+Connection ~ 1450 8700
+Wire Wire Line
+	1450 8700 1450 8750
+Wire Wire Line
+	4850 9550 5100 9550
+$Comp
+L Device:C C22
+U 1 1 60B6548E
+P 5100 9700
+F 0 "C22" H 4800 9750 50  0000 L CNN
+F 1 "100n" H 4800 9650 50  0000 L CNN
+F 2 "" H 5138 9550 50  0001 C CNN
+F 3 "~" H 5100 9700 50  0001 C CNN
+	1    5100 9700
+	1    0    0    -1
+$EndComp
+Connection ~ 5100 9550
+Wire Wire Line
+	5100 9550 5350 9550
+Wire Wire Line
+	5100 9850 5100 9900
+$Comp
+L power:GND #PWR05
+U 1 1 60B7E9A3
+P 5100 9900
+F 0 "#PWR05" H 5100 9650 50  0001 C CNN
+F 1 "GND" H 5105 9727 50  0000 C CNN
+F 2 "" H 5100 9900 50  0001 C CNN
+F 3 "" H 5100 9900 50  0001 C CNN
+	1    5100 9900
+	1    0    0    -1
+$EndComp
 $EndSCHEMATC

Commit message: Encore
Parts:
- R16: value R -> 10k
Changed lines of the file:
@@
 P 2250 8500
 F 0 "R16" H 2320 8546 50  0000 L CNN
-F 1 "R" H 2320 8455 50  0000 L CNN
+F 1 "10k" H 2320 8455 50  0000 L CNN
 F 2 "" V 2180 8500 50  0001 C CNN
 F 3 "~" H 2250 8500 50  0001 C CNN
